File: 858D.kicad_sch (KiCad schematic)
At the start: 70 parts, among them J2 Transformer, J3 Conn_01x02, K1 SRD-12VDC-SL-C, M1 Fan, Q1 TIP122, Q2 MMBT3904, Q3 MMBT3904, Q4 MMBT3904, SW1 SW_Reed, SW2 SW_SPST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

Commit message: Add files via upload
Connections:
- net Reed: now also R27.2; no longer C15.2, R22.1, R23.1
- net Thermocouple: now also C15.2, R22.1, R23.1; no longer R27.2
Changed lines of the file:
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@@
-    (stroke (width 0) (type default))
-  )
-  (wire (pts (xy 52.07 52.705) (xy 54.61 52.705))
     (stroke (width 0) (type default))
   )
@@
     (stroke (width 0) (type default))
   )
-  (wire (pts (xy 71.755 17.78) (xy 68.58 17.78))
-    (stroke (width 0) (type default))
-  )
   (wire (pts (xy 114.935 136.525) (xy 128.27 136.525))
     (stroke (width 0) (type default))
@@
     (stroke (width 0) (type default))
   )
+  (wire (pts (xy 67.945 17.78) (xy 71.755 17.78))
+    (stroke (width 0) (type default))
+  )
   (wire (pts (xy 226.695 22.225) (xy 226.695 26.035))
     (stroke (width 0) (type default))
@@
   )
   (wire (pts (xy 59.69 52.705) (xy 54.61 52.705))
+    (stroke (width 0) (type default))
+  )
+  (wire (pts (xy 50.8 52.705) (xy 54.61 52.705))
     (stroke (width 0) (type default))
   )
@@
     )
   )
-  (global_label "Reed" (shape input) (at 52.07 52.705 180) (fields_autoplaced)
+  (global_label "Reed" (shape input) (at 67.945 17.78 180) (fields_autoplaced)
     (effects (font (size 1.27 1.27) (color 0 0 255 1)) (justify right))
-    (property "Intersheetrefs" "${INTERSHEET_REFS}" (at 44.568 52.705 0)
+    (property "Intersheetrefs" "${INTERSHEET_REFS}" (at 60.443 17.78 0)
       (effects (font (size 1.27 1.27)) (justify right) hide)
     )
@@
     )
   )
-  (global_label "Thermocouple" (shape input) (at 68.58 17.78 180) (fields_autoplaced)
+  (global_label "Thermocouple" (shape input) (at 50.8 52.705 180) (fields_autoplaced)
     (effects (font (size 1.27 1.27) (color 255 0 0 1)) (justify right))
-    (property "Intersheetrefs" "${INTERSHEET_REFS}" (at 52.5511 17.78 0)
-      (effects (font (size 1.27 1.27)) (justify right) hide)
-    )
+    (property "Intersheetrefs" "${INTERSHEET_REFS}" (at 34.7711 52.705 0)
+      (effects (font (size 1.27 1.27)) (justify right) hide)
+    )
